File: Rendition 1/UGV_Board.kicad_pcb (KiCad board)
At the start: 2 copper layers, 43 parts, among them J1 I2C_EXPANSION, J2 Debug Header, J3 ESP_Header, J4 RFLCTR_Header, J5 RFLCTL_Header, J6 IMU_Daughter_Header, J7 Conn_01x02_Female, J8 Conn_01x02_Female, SW1 SW_MCU_EN, SW2 SW_PICO_RST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

Commit message: Completed KiKad First Draft
Parts:
- moved R7 51.9 mm to (139.7, 132.8)
- moved J4 33.2 mm to (139.7, 137.2), turned to 0 degrees
- moved C3 31.0 mm to (144.8, 144.8), turned to 0 degrees
- moved SW1 27.4 mm to (129.5, 104.1), turned to 180 degrees
- moved U2 24.1 mm to (132.1, 115.0), turned to -90 degrees
- moved RV3 23.0 mm to (132.1, 127.0), turned to 180 degrees
- moved L1 21.8 mm to (144.8, 139.7), turned to -90 degrees
- moved R13 20.5 mm to (139.7, 129.5), turned to 180 degrees
- moved J8 17.8 mm to (139.7, 104.1), turned to 90 degrees
- moved SW2 17.8 mm to (125.2, 124.2)
- moved R8 16.3 mm to (132.1, 137.2), turned to 0 degrees
- moved R9 16.1 mm to (132.1, 139.7), turned to 0 degrees
- moved R10 15.5 mm to (132.1, 144.8), turned to 0 degrees
- moved R4 15.5 mm to (118.4, 109.2), turned to 0 degrees
- moved R6 15.5 mm to (119.4, 111.8), turned to 0 degrees
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Routing:
- net Net-(R13-Pad2): track 12.7 -> 64.9 mm
- net Net-(J5-Pad3): track 8.28 -> 43.4 mm
- net Net-(J4-Pad1): track 51.3 -> 83.1 mm
- net Net-(C4-Pad1): track 39.8 -> 17.1 mm
- net Net-(C3-Pad2): track 3.74 -> 26.0 mm
- net Net-(J5-Pad1): track 46.7 -> 67.2 mm
- net +6V: track 79.5 -> 96.9 mm
- net Net-(R3-Pad2): track 17.3 -> 5.24 mm
- net Net-(C3-Pad1): track 15.8 -> 26.9 mm
- net Net-(J8-Pad2): track 5.46 -> 16.3 mm
- net Net-(J7-Pad1): track 5.43 -> 15.7 mm
- net Net-(J8-Pad1): track 6.84 -> 16.6 mm
- net Net-(D4-Pad1): track 14.3 -> 5.61 mm
- net SDA: track 95.4 -> 86.7 mm
- net Net-(SW1-Pad1): track 5.08 -> 13.2 mm
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