File: _autosave-UGV_Board.kicad_sch (KiCad schematic)
At the start: 45 parts, among them J1 I2C_EXPANSION, J2 Debug Header, J3 ESP_Header, J4 RFLCTR_Header, J5 RFLCTL_Header, J6 IMU_Daughter_Header, J7 Conn_01x02_Female, J8 Conn_01x02_Female, SW1 SW_MCU_EN, SW2 SW_PICO_RST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

Commit message: Rev 1 Final
Parts:
- gave numbers to parts that had none: 1
Changed lines of the file:
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@@
   (symbol (lib_id "Connector:Conn_01x02_Female") (at 443.9619 125.6615 0) (unit 1)
     (in_bom yes) (on_board yes)
-    (property "Reference" "J?" (id 0) (at 445.2319 125.6614 0)
+    (property "Reference" "J9" (id 0) (at 445.2319 125.6614 0)
       (effects (font (size 1.27 1.27)) (justify left))
     )
@@
   (symbol (lib_id "power:GND") (at 432.9043 129.5787 0) (unit 1)
     (in_bom yes) (on_board yes)
-    (property "Reference" "#PWR?" (id 0) (at 432.9043 135.9287 0)
+    (property "Reference" "#PWR0139" (id 0) (at 432.9043 135.9287 0)
       (effects (font (size 1.27 1.27)) hide)
     )
@@
   (symbol (lib_id "power:+7.5V") (at 432.9539 123.083 90) (unit 1)
     (in_bom yes) (on_board yes)
-    (property "Reference" "#PWR?" (id 0) (at 436.7639 123.083 0)
+    (property "Reference" "#PWR0138" (id 0) (at 436.7639 123.083 0)
       (effects (font (size 1.27 1.27)) hide)
     )
@@
       (reference "#PWR0137") (unit 1) (value "+3.3V") (footprint "")
     )
+    (path "/dc43a708-df8c-4a6b-a99f-7b0d9d026ff5"
+      (reference "#PWR0138") (unit 1) (value "+7.5V") (footprint "")
+    )
     (path "/d099c49c-0d3c-4d8f-8b16-ad1a9bb31217"
-      (reference "#PWR?") (unit 1) (value "GND") (footprint "")
-    )
-    (path "/dc43a708-df8c-4a6b-a99f-7b0d9d026ff5"
-      (reference "#PWR?") (unit 1) (value "+7.5V") (footprint "")
+      (reference "#PWR0139") (unit 1) (value "GND") (footprint "")
     )
     (path "/8e5869e2-bbd2-4bca-8704-5fa8462ff71f"
@@
     )
     (path "/1fcaef59-27d4-4242-8360-ac5b1e33e3e7"
-      (reference "J?") (unit 1) (value "Battery Header") (footprint "Connector_PinSocket_2.54mm:PinSocket_1x02_P2.54mm_Vertical")
+      (reference "J9") (unit 1) (value "Battery Header") (footprint "Connector_PinSocket_2.54mm:PinSocket_1x02_P2.54mm_Vertical")
     )
     (path "/8e1f62bc-e92b-4dd3-93ab-1ffac33da743"
