File: UGV_Board.kicad_pcb (KiCad board)
At the start: 2 copper layers, 46 parts, among them J1 I2C_EXPANSION, J2 Debug Header, J3 ESP_Header, J4 RFLCTR_Header, J5 RFLCTL_Header, J6 IMU_Daughter_Header, J7 Conn_01x02_Female, J8 Conn_01x02_Female, J9 Battery Header, SW1 SW_MCU_EN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

Commit message: v2 schematic
Parts:
- removed C1: 10uF, Capacitor_SMD:C_1206_3216Metric_Pad1.33x1.80mm_HandSolder
- removed C2: 22uF, Capacitor_SMD:C_1206_3216Metric_Pad1.33x1.80mm_HandSolder
- removed C3: 100nF, Capacitor_SMD:C_1206_3216Metric_Pad1.33x1.80mm_HandSolder
- removed C5: 22 uF, Capacitor_SMD:C_1206_3216Metric_Pad1.33x1.80mm_HandSolder
- removed L1: 4.7uH, Inductor_SMD:L_1210_3225Metric_Pad1.42x2.65mm_HandSolder
- removed R10, R7, R8, R9: 220, Resistor_SMD:R_1206_3216Metric_Pad1.30x1.75mm_HandSolder
- removed R13: 10k, Resistor_SMD:R_1206_3216Metric_Pad1.30x1.75mm_HandSolder
- removed R14, R15: 1k, Resistor_SMD:R_1206_3216Metric_Pad1.30x1.75mm_HandSolder
- removed the R2 at (193.7, 82.9)
- removed RV1, RV2, RV3: R_Potentiometer, Potentiometer_SMD:Potentiometer_Bourns_TC33X_Vertical
- removed U3: LM393, Package_DIP:DIP-8_W7.62mm_LongPads
- removed U4: BD63565EFV-E2, Drivers_3rdParty:BD63565EFV-E2
- removed U5: AP62200WU-7, SMPS_3rdParty:AP62200WU-7
- added J9: Buck Input, Connector_PinSocket_2.54mm:PinSocket_1x02_P2.54mm_Vertical, F.Cu at (168.1, 132.1)
- D2, D3, D4: footprint LED_SMD:LED_2010_5025Metric_Pad1.52x2.65mm_HandSolder -> LED_THT:LED_D5.0mm
- J4: value RFLCTR_Header -> ENCR_Header
- J5: value RFLCTL_Header -> ENCL_Header
- J7: value Conn_01x02_Female -> MotorL
- J8: value Conn_01x02_Female -> MotorR
- moved J7 62.9 mm to (172.7, 132.1), turned to 0 degrees
- moved J8 52.2 mm to (177.3, 132.1), turned to 0 degrees
- renumbered J9 to J10
Connections:
- J4 pad 1: Net-(J4-Pad1) -> ESP_GND
- J4 pad 2: ESP_3.3V -> ENCRA_SIG
- J4 pad 3: Net-(J4-Pad3) -> ENCRB_SIG
- J5 pad 1: Net-(J5-Pad1) -> ESP_GND
- J5 pad 2: ESP_3.3V -> ENCLA_SIG
- J5 pad 3: Net-(J5-Pad3) -> ENCLB_SIG
- J6 pad 5: MAG_DRDY -> CSB
- J6 pad 6: MAG_INT -> INT1
- J6 pad 7: IMU_INT1 -> INT2
- J6 pad 8: IMU_INT2 -> (no net)
- J7 pad 1: Net-(J7-Pad1) -> MOTORLB_SIG
- J7 pad 2: Net-(J7-Pad2) -> MOTORLA_SIG
- J8 pad 1: Net-(J8-Pad1) -> MOTORRB_SIG
- J8 pad 2: Net-(J8-Pad2) -> MOTORRA_SIG
- U1 pad 10: MAG_INT -> CSB
- U1 pad 11: IMU_INT1 -> INT1
- U1 pad 12: IMU_INT2 -> INT2
- U1 pad 19: ENCL_SIG -> ENCLA_SIG
- U1 pad 20: ENCR_SIG -> ENCLB_SIG
- U1 pad 21: unconnected-(U1-Pad21) -> ENCRA_SIG
- U1 pad 22: unconnected-(U1-Pad22) -> ENCRB_SIG
- U1 pad 9: MAG_DRDY -> unconnected-(U1-Pad9)
Routing:
- net (no net): track 0.00 -> 190.7 mm, vias 0 -> 2
- net INT2: track 0.00 -> 111.5 mm, vias 0 -> 1
- net ESP_GND: track 348.1 -> 437.0 mm
- net Net-(J5-Pad1): track 88.9 -> 0.00 mm
- net MAG_INT: track 57.3 -> 0.00 mm, vias 1 -> 0
- net INT1: track 0.00 -> 57.3 mm, vias 0 -> 1
- net IMU_INT1: track 56.0 -> 0.00 mm, vias 1 -> 0
- net IMU_INT2: track 55.5 -> 0.00 mm, vias 1 -> 0
- net MAG_DRDY: track 52.2 -> 0.00 mm, vias 1 -> 0
- net CSB: track 0.00 -> 52.2 mm, vias 0 -> 1
- net Net-(R13-Pad2): track 48.5 -> 0.00 mm
- net +6V: track 46.6 -> 0.00 mm
- net ESP_3.3V: track 259.2 -> 291.9 mm
- net Net-(C3-Pad1): track 29.0 -> 0.00 mm, vias 2 -> 0
- net ENCLB_SIG: track 0.00 -> 28.2 mm
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
Commit message: KiKAD Rev 2 Feb 17
Parts:
- moved SW1 96.9 mm to (199.9, 63.0), turned to -90 degrees
- moved J7 80.7 mm to (131.1, 63.0)
- moved J8 80.2 mm to (136.7, 63.0)
- moved J10 64.0 mm to (199.6, 69.6), turned to 0 degrees
- moved J5 62.8 mm to (176.5, 63.0)
- moved U2 49.9 mm to (172.2, 73.7)
- moved R6 40.2 mm to (194.6, 112.3), turned to 180 degrees
- moved D4 38.6 mm to (182.9, 99.3), turned to 90 degrees
- moved R5 34.2 mm to (194.6, 108.7), turned to 180 degrees
- moved D3 29.2 mm to (182.9, 89.7), turned to 90 degrees
- moved R4 28.2 mm to (194.6, 105.2), turned to 180 degrees
- moved SW2 28.0 mm to (170.5, 90.6), turned to 90 degrees
- moved J6 27.1 mm to (131.1, 85.6)
- moved R11 26.9 mm to (137.2, 80.3)
- moved D2 25.6 mm to (182.9, 78.5), turned to 90 degrees
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Routing:
- net ESP_GND: track 437.0 -> 214.8 mm, vias 1 -> 0
- net (no net): track 190.7 -> 0.00 mm, vias 2 -> 0
- net ESP_3.3V: track 291.9 -> 130.0 mm, vias 4 -> 0
- net INT2: track 111.5 -> 15.8 mm, vias 1 -> 0
- net ESP_TX: track 6.99 -> 75.9 mm, vias 1 -> 2
- net ESP_RX: track 6.74 -> 72.9 mm, vias 1 -> 3
- net ENCRA_SIG: track 0.00 -> 60.9 mm, vias 0 -> 1
- net ENCRB_SIG: track 0.00 -> 60.3 mm, vias 0 -> 1
- net ENCLA_SIG: track 7.90 -> 65.0 mm
- net ENCLB_SIG: track 28.2 -> 79.4 mm, vias 0 -> 1
- net SCL: track 73.6 -> 28.5 mm, vias 2 -> 0
- net MOTORRB_SIG: track 13.5 -> 58.4 mm
- net INT1: track 57.3 -> 16.3 mm, vias 1 -> 0
- net MOTORRA_SIG: track 13.5 -> 53.6 mm
- net SDA: track 80.1 -> 41.1 mm, vias 1 -> 0
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
Commit message: final
Parts:
- J6: footprint Connector_PinSocket_2.54mm:PinSocket_1x08_P2.54mm_Vertical -> Connector_PinHeader_2.54mm:PinHeader_1x07_P2.54mm_Vertical
Connections:
- J9 pad 2: unconnected-(J9-Pad2) -> +7.5V
Routing:
- net +7.5V: track 24.9 -> 88.0 mm
Other:
- board outline added: 75.5 x 58 mm
