File: UGV_Board.kicad_sch (KiCad schematic)
At the start: 28 parts, among them J1 I2C_EXPANSION, J10 Battery Header, J2 Debug Header, J3 ESP_Header, J4 ENCR_Header, J5 ENCL_Header, J6 IMU_Daughter_Header, J7 MotorL, J8 MotorR, J9 Buck Input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

Commit message: final
Parts:
- J6: footprint Connector_PinSocket_2.54mm:PinSocket_1x08_P2.54mm_Vertical -> Connector_PinHeader_2.54mm:PinHeader_1x07_P2.54mm_Vertical
Connections:
- net +7.5V: now also J9.2 (Pin_2)
Changed lines of the file:
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@@
     (stroke (width 0) (type default) (color 0 0 0 0))
   )
-  (wire (pts (xy 388.62 143.51) (xy 388.62 146.05))
+  (wire (pts (xy 388.62 140.97) (xy 386.08 140.97))
+    (stroke (width 0) (type default) (color 0 0 0 0))
+  )
+  (wire (pts (xy 388.62 140.97) (xy 388.62 146.05))
     (stroke (width 0) (type default) (color 0 0 0 0))
   )
@@
     (property "Reference" "J6" (id 0) (at 335.28 226.06 90))
     (property "Value" "IMU_Daughter_Header" (id 1) (at 335.28 228.6 90))
-    (property "Footprint" "Connector_PinSocket_2.54mm:PinSocket_1x08_P2.54mm_Vertical" (id 2) (at 334.01 231.14 0)
+    (property "Footprint" "Connector_PinHeader_2.54mm:PinHeader_1x07_P2.54mm_Vertical" (id 2) (at 334.01 231.14 0)
       (effects (font (size 1.27 1.27)) hide)
     )
@@
     (pin "2")
   )
-  (symbol (lib_id "power:+7.5V") (at 388.6696 143.4715 90) (unit 1)
-    (in_bom yes) (on_board yes)
-    (property "Reference" "#PWR0114" (id 0) (at 392.4796 143.4715 0)
-      (effects (font (size 1.27 1.27)) hide)
-    )
-    (property "Value" "+7.5V" (id 1) (at 379.7796 143.4715 90)
+  (symbol (lib_id "power:+7.5V") (at 386.08 140.97 90) (unit 1)
+    (in_bom yes) (on_board yes)
+    (property "Reference" "#PWR0114" (id 0) (at 389.89 140.97 0)
+      (effects (font (size 1.27 1.27)) hide)
+    )
+    (property "Value" "+7.5V" (id 1) (at 377.19 140.97 90)
       (effects (font (size 1.27 1.27)) (justify right))
     )
-    (property "Footprint" "" (id 2) (at 388.6696 143.4715 0)
-      (effects (font (size 1.27 1.27)) hide)
-    )
-    (property "Datasheet" "" (id 3) (at 388.6696 143.4715 0)
+    (property "Footprint" "" (id 2) (at 386.08 140.97 0)
+      (effects (font (size 1.27 1.27)) hide)
+    )
+    (property "Datasheet" "" (id 3) (at 386.08 140.97 0)
       (effects (font (size 1.27 1.27)) hide)
     )
@@
     )
     (path "/3003f17c-94b7-4548-9672-5693c4f2161a"
-      (reference "J6") (unit 1) (value "IMU_Daughter_Header") (footprint "Connector_PinSocket_2.54mm:PinSocket_1x08_P2.54mm_Vertical")
+      (reference "J6") (unit 1) (value "IMU_Daughter_Header") (footprint "Connector_PinHeader_2.54mm:PinHeader_1x07_P2.54mm_Vertical")
     )
     (path "/d2087407-0a85-45c3-b530-8a0814cb9106"
