File: Rendition 3/UGV_Board.kicad_pcb (KiCad board)
At the start: 2 copper layers, 46 parts, among them J1 I2C_EXPANSION, J2 Debug Header, J3 ESP_Header, J4 RFLCTR_Header, J5 RFLCTL_Header, J6 IMU_Daughter_Header, J7 Conn_01x02_Female, J8 Conn_01x02_Female, J9 Battery Header, SW1 SW_MCU_EN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

Commit message: Rev 1 Final
Parts:
- moved D3 135.3 mm to (81.3, 121.9), turned to -90 degrees
- moved J3 133.4 mm to (81.3, 139.7), turned to 180 degrees
- moved SW3 129.4 mm to (81.3, 99.1), turned to 0 degrees
- moved J4 128.4 mm to (115.6, 160.0)
- moved R5 120.6 mm to (81.3, 114.3), turned to -90 degrees
- moved R9 120.2 mm to (127.0, 154.9), turned to -90 degrees
- moved RV2 112.9 mm to (83.8, 144.8)
- moved U3 110.7 mm to (80.0, 158.8)
- moved D2 98.3 mm to (116.8, 116.6), turned to 90 degrees
- moved J5 98.0 mm to (123.2, 155.0)
- moved D4 97.0 mm to (121.9, 114.3), turned to 180 degrees
- moved R7 95.9 mm to (94.0, 157.5), turned to 180 degrees
- moved R6 91.5 mm to (121.9, 127.0), turned to 180 degrees
- moved R4 88.2 mm to (120.9, 124.5), turned to 180 degrees
- moved J1 86.6 mm to (130.8, 157.5), turned to 90 degrees
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Routing:
- net Net-(J4-Pad1): track 0.11 -> 51.3 mm
- net MAG_INT: track 57.3 -> 6.75 mm, vias 1 -> 0
- net IMU_INT1: track 56.0 -> 6.75 mm, vias 1 -> 0
- net IMU_INT2: track 55.5 -> 6.75 mm, vias 1 -> 0
- net ESP_GPIO0: track 14.0 -> 62.7 mm
- net MAG_DRDY: track 52.2 -> 6.75 mm, vias 1 -> 0
- net ESP_TX: track 6.99 -> 49.4 mm, vias 1 -> 0
- net Net-(J5-Pad1): track 88.9 -> 46.7 mm
- net Net-(SW1-Pad1): track 44.9 -> 5.08 mm
- net Net-(R13-Pad2): track 48.5 -> 12.7 mm
- net ESP_RX: track 6.74 -> 42.0 mm, vias 1 -> 0
- net +6V: track 46.6 -> 79.5 mm
- net Net-(C4-Pad1): track 11.4 -> 39.8 mm
- net Net-(RV1-Pad2): track 0.00 -> 23.8 mm
- net MOTORLB_SIG: track 20.7 -> 0.00 mm
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