File: Rendition 4/UGV_Board.kicad_pcb (KiCad board)
At the start: 2 copper layers, 46 parts, among them J1 I2C_EXPANSION, J2 Debug Header, J3 ESP_Header, J4 RFLCTR_Header, J5 RFLCTL_Header, J6 IMU_Daughter_Header, J7 Conn_01x02_Female, J8 Conn_01x02_Female, J9 Battery Header, SW1 SW_MCU_EN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

Commit message: Rev 1 Final
Parts:
- moved R8 26.0 mm to (200.7, 105.1)
- moved D2 7.29 mm to (201.1, 81.7)
- moved D3 7.29 mm to (201.1, 76.4)
- moved R4 7.29 mm to (188.0, 77.9)
- moved R6 7.29 mm to (187.9, 73.0)
- moved SW3 7.29 mm to (203.0, 89.2)
- moved D4 7.29 mm to (201.2, 71.3)
- moved R5 7.29 mm to (187.9, 75.4)
- moved R2 7.29 mm to (186.5, 83.8)
- moved R9 5.81 mm to (201.0, 67.0)
- moved RV2 4.12 mm to (193.0, 109.2)
- moved J4 2.24 mm to (195.6, 61.0)
- moved R7 2.05 mm to (180.3, 111.8)
- moved U3 1.94 mm to (175.3, 105.8)
- moved J3 1.61 mm to (190.2, 62.9)
Routing:
- net ESP_GND: track 348.1 -> 413.1 mm
- net Net-(J4-Pad1): track 0.11 -> 59.5 mm
- net ESP_TX: track 6.99 -> 60.3 mm
- net ESP_3.3V: track 259.2 -> 310.4 mm
- net ENCR_SIG: track 21.3 -> 64.8 mm
- net ESP_RX: track 6.74 -> 48.0 mm
- net ENCL_SIG: track 7.90 -> 45.2 mm
- net Net-(C4-Pad1): track 11.4 -> 32.7 mm
- net ESP_RST: track 26.8 -> 46.1 mm
- net Net-(J5-Pad1): track 88.9 -> 107.8 mm
- net Net-(RV2-Pad2): track 0.00 -> 16.7 mm
- net ESP_GPIO0: track 14.0 -> 27.1 mm
- net Net-(RV1-Pad2): track 0.00 -> 11.8 mm
- net ESP_GPIO2: track 18.6 -> 27.1 mm
- net Net-(D1-Pad2): track 15.1 -> 22.2 mm
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
Commit message: final changes
Parts:
- J7: value Conn_01x02_Female -> Motor Left
- J8: value Conn_01x02_Female -> Motor Right
Other:
- board outline added: 110 x 70 mm
Changed lines of the file:
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@@
     (property "Sheetname" "")
     (attr through_hole)
-    (fp_text reference "SW1" (at 0.4 -2.7) (layer "F.SilkS")
-      (effects (font (size 1 1) (thickness 0.15)))
-    )
-    (fp_text value "SW_MCU_EN" (at -6 -2.7) (layer "F.SilkS")
+    (fp_text reference "SW1" (at 4.3 1.3) (layer "Dwgs.User")
+      (effects (font (size 1 1) (thickness 0.15)))
+    )
+    (fp_text value "SW_MCU_EN" (at -2.4 -3) (layer "F.SilkS")
       (effects (font (size 1 1) (thickness 0.15)))
     )
@@
       (effects (font (size 1 1) (thickness 0.15)))
     )
-    (fp_text value "10k" (at 0 1.82 90) (layer "F.Fab")
+    (fp_text value "10k" (at 0 1.82 90) (layer "F.SilkS")
       (effects (font (size 1 1) (thickness 0.15)))
     )
@@
       (effects (font (size 1 1) (thickness 0.15)))
     )
-    (fp_text value "220" (at 0 1.82 90) (layer "F.Fab")
+    (fp_text value "220" (at 0 2.14 90) (layer "F.SilkS")
       (effects (font (size 1 1) (thickness 0.15)))
     )
@@
       (effects (font (size 1 1) (thickness 0.15)))
     )
-    (fp_text value "330" (at 4.15 0) (layer "F.Fab")
+    (fp_text value "330" (at 4.15 0) (layer "F.SilkS")
       (effects (font (size 1 1) (thickness 0.15)))
     )
@@
       (effects (font (size 1 1) (thickness 0.15)))
     )
-    (fp_text value "Conn_01x02_Female" (at -2.66 7.04 180) (layer "F.SilkS")
+    (fp_text value "Motor Left" (at -2.66 7.04 180) (layer "F.SilkS")
       (effects (font (size 1 1) (thickness 0.15)))
     )
@@
       (effects (font (size 1 1) (thickness 0.15)))
     )
-    (fp_text value "1k" (at -5.07 -1.3 90) (layer "F.Fab")
+    (fp_text value "1k" (at -3.95 0.1 180) (layer "F.SilkS")
       (effects (font (size 1 1) (thickness 0.15)))
     )
@@
       (effects (font (size 1 1) (thickness 0.15)))
     )
-    (fp_text value "Conn_01x02_Female" (at 3.175 -5.35) (layer "F.SilkS")
+    (fp_text value "Motor Right" (at 3.175 -3.25) (layer "F.SilkS")
       (effects (font (size 1 1) (thickness 0.15)))
     )
@@
       (effects (font (size 1 1) (thickness 0.15)))
     )
-    (fp_text value "330" (at 0 1.82) (layer "F.Fab")
+    (fp_text value "330" (at -0.2 -3.3) (layer "F.SilkS")
       (effects (font (size 1 1) (thickness 0.15)))
     )
@@
       (effects (font (size 1 1) (thickness 0.15)))
     )
-    (fp_text value "220" (at -0.15 1.6 90) (layer "F.Fab")
+    (fp_text value "220" (at -1.24 2.56 90) (layer "F.SilkS")
       (effects (font (size 1 1) (thickness 0.15)))
     )
@@
     (property "Sheetname" "")
     (attr smd)
-    (fp_text reference "R2" (at 0 -1.82) (layer "F.SilkS")
-      (effects (font (size 1 1) (thickness 0.15)))
-    )
-    (fp_text value "330" (at 0 1.82) (layer "F.Fab")
+    (fp_text reference "R2" (at 2.8 -1.82) (layer "F.SilkS")
+      (effects (font (size 1 1) (thickness 0.15)))
+    )
+    (fp_text value "330" (at -0.1 -1.9) (layer "F.SilkS")
       (effects (font (size 1 1) (thickness 0.15)))
     )
@@
     (property "Sheetname" "")
     (attr smd)
-    (fp_text reference "R1" (at 0 -1.82) (layer "F.SilkS")
-      (effects (font (size 1 1) (thickness 0.15)))
-    )
-    (fp_text value "330" (at 0 1.82) (layer "F.Fab")
+    (fp_text reference "R1" (at 2.8 1.8) (layer "F.SilkS")
+      (effects (font (size 1 1) (thickness 0.15)))
+    )
+    (fp_text value "330" (at 0 1.82) (layer "F.SilkS")
       (effects (font (size 1 1) (thickness 0.15)))
     )
@@
     (fp_text value "SC0915" (at 0.14738 4.27357) (layer "F.SilkS")
       (effects (font (size 1 1) (thickness 0.15)))
-    )
-    (fp_text user "Copyright 2021 Accelerated Designs. All rights reserved." (at 37.8625 -27.86) (layer "Cmts.User")
-      (effects (font (size 0.127 0.127) (thickness 0.002)))
     )
     (fp_line (start -3.67284 25.6286) (end -10.6299 25.6286) (layer "F.SilkS") (width 0.12))
@@
       (effects (font (size 1 1) (thickness 0.15)))
     )
-    (fp_text value "330" (at 4.12 -0.06) (layer "F.Fab")
+    (fp_text value "330" (at 4.12 -0.06) (layer "F.SilkS")
       (effects (font (size 1 1) (thickness 0.15)))
     )
@@
       (effects (font (size 1 1) (thickness 0.15)))
     )
-    (fp_text value "330" (at 4.05 -0.1) (layer "F.Fab")
+    (fp_text value "330" (at 4.05 -0.1) (layer "F.SilkS")
       (effects (font (size 1 1) (thickness 0.15)))
     )
@@
       (effects (font (size 1 1) (thickness 0.15)))
     )
-    (fp_text value "1k" (at 0 1.82) (layer "F.Fab")
+    (fp_text value "1k" (at 0 1.82) (layer "F.SilkS")
       (effects (font (size 1 1) (thickness 0.15)))
     )
@@
     (property "Sheetname" "")
     (attr smd)
-    (fp_text reference "R12" (at 0 -1.82 90) (layer "F.SilkS")
-      (effects (font (size 1 1) (thickness 0.15)))
-    )
-    (fp_text value "10k" (at 0 1.82 90) (layer "F.Fab")
+    (fp_text reference "R12" (at 3.15 0.2 180) (layer "F.SilkS")
+      (effects (font (size 1 1) (thickness 0.15)))
+    )
+    (fp_text value "10k" (at 0.35 2.1 90) (layer "F.SilkS")
       (effects (font (size 1 1) (thickness 0.15)))
     )
@@
       (effects (font (size 1 1) (thickness 0.15)))
     )
-    (fp_text value "SW_PICO_RST" (at 3.75 6.7) (layer "F.Fab")
+    (fp_text value "SW_PICO_RST" (at 3.75 6.7) (layer "F.SilkS")
       (effects (font (size 1 1) (thickness 0.15)))
     )
@@
       (effects (font (size 1 1) (thickness 0.15)))
     )
-    (fp_text value "220" (at -0.1 2.3 90) (layer "F.Fab")
+    (fp_text value "220" (at -0.1 2.3 90) (layer "F.SilkS")
       (effects (font (size 1 1) (thickness 0.15)))
     )
@@
       (effects (font (size 1 1) (thickness 0.15)))
     )
-    (fp_text value "R_Small_US" (at 0 1.82 -270) (layer "F.Fab")
+    (fp_text value "R_Small_US" (at 0.38 2.969423 -270) (layer "F.Fab")
       (effects (font (size 1 1) (thickness 0.15)))
     )
@@
       (effects (font (size 1 1) (thickness 0.15)))
     )
-    (fp_text value "1uF" (at 0 1.85) (layer "F.Fab")
+    (fp_text value "1uF" (at 0 1.85) (layer "F.SilkS")
       (effects (font (size 1 1) (thickness 0.15)))
     )
@@
     )
   )
+  (gr_rect (start 99 51.6) (end 209 121.6) (layer "Edge.Cuts") (width 0.1) (fill none))
   (segment (start 175.6 92.9) (end 170.25 98.25) (width 0.25) (layer "F.Cu") (net 1))
   (segment (start 170.25 98.25) (end 170.25 98.6) (width 0.25) (layer "F.Cu") (net 1))
@@
   (segment (start 127.065 101.271998) (end 127.065 114.631701) (width 0.25) (layer "F.Cu") (net 14))
   (segment (start 190.2 62.89) (end 190.2 69.148173) (width 0.25) (layer "F.Cu") (net 14))
+  (segment (start 128.365 85.185) (end 130.285 85.185) (width 0.25) (layer "F.Cu") (net 14))
   (segment (start 127.065 114.631701) (end 125.396701 116.3) (width 0.25) (layer "F.Cu") (net 14))
   (segment (start 192.388173 66.96) (end 190.2 69.148173) (width 0.25) (layer "F.Cu") (net 14))
+  (segment (start 130.905 85.375978) (end 130.905 86.405) (width 0.25) (layer "F.Cu") (net 14))
   (segment (start 148.5824 63.03643) (end 161.94272 63.03643) (width 0.25) (layer "F.Cu") (net 14))
   (segment (start 175.97 58.71) (end 169.47 58.71) (width 0.25) (layer "F.Cu") (net 14))
@@
   (segment (start 127.725 57.275) (end 126.8023 58.1977) (width 0.25) (layer "F.Cu") (net 14))
   (segment (start 127.624626 69.7) (end 129.339751 71.415125) (width 0.25) (layer "F.Cu") (net 14))
+  (segment (start 130.714511 85.185489) (end 130.905 85.375978) (width 0.25) (layer "F.Cu") (net 14))
   (segment (start 138.1 64.3) (end 147.31883 64.3) (width 0.25) (layer "F.Cu") (net 14))
   (segment (start 190.2 69.148173) (end 186.368173 72.98) (width 0.25) (layer "F.Cu") (net 14))
   (segment (start 116.9 69.7) (end 127.624626 69.7) (width 0.25) (layer "F.Cu") (net 14))
+  (segment (start 130.285 85.185) (end 130.285489 85.185489) (width 0.25) (layer "F.Cu") (net 14))
   (segment (start 120.3575 96.52) (end 120.3575 99.06) (width 0.25) (layer "F.Cu") (net 14))
+  (segment (start 130.285489 85.185489) (end 130.714511 85.185489) (width 0.25) (layer "F.Cu") (net 14))
   (segment (start 127.915002 87.984998) (end 128.365 87.535) (width 0.25) (layer "F.Cu") (net 14))
   (segment (start 180.34 113.31) (end 182.88 110.77) (width 0.25) (layer "F.Cu") (net 14))
   (segment (start 123.315 85.185) (end 128.365 85.185) (width 0.25) (layer "F.Cu") (net 14))
   (segment (start 132.39 94.553399) (end 130.589999 94.553399) (width 0.25) (layer "F.Cu") (net 14))
-  (segment (start 128.365 85.185) (end 130.905 85.185) (width 0.25) (layer "F.Cu") (net 14))
   (segment (start 203.019423 89.17) (end 196.119423 82.27) (width 0.25) (layer "F.Cu") (net 14))
   (segment (start 175.6 89.075) (end 169.925 83.4) (width 0.25) (layer "F.Cu") (net 14))
@@
   (segment (start 186.368173 72.98) (end 186.368173 75.4) (width 0.25) (layer "F.Cu") (net 14))
   (segment (start 119.2625 89.2375) (end 123.315 85.185) (width 0.25) (layer "F.Cu") (net 14))
-  (segment (start 130.905 85.185) (end 130.905 86.405) (width 0.25) (layer "F.Cu") (net 14))
   (segment (start 182.88 110.77) (end 182.88 105.825) (width 0.25) (layer "F.Cu") (net 14))
   (segment (start 186.368173 75.4) (end 186.388173 75.42) (width 0.25) (layer "F.Cu") (net 14))
